Commit message: 添加ros2_control.xacro

File: urdf/aubo_i10.urdf.xacro (robot description, xacro)
@@ -1,209 +1,267 @@
 <?xml version="1.0"?>
 <robot name="aubo_i10"
-  xmlns:xacro="http://wiki.ros.org/xacro">
-  <dh_type type="modified"/>
-  <safety_para singularity_consistent="0.02 0.01 10 0.2 0.045 10"/>
-  <friction_coeff value="0.65"/>
-  <link name="base_link">
-    <inertial>
-      <origin xyz="0.000136 0.001601 0.018986" rpy="0 0 0" />
-      <mass value="2.592" />
-      <inertia ixx="0.008524" ixy="-0.000001" ixz="-0.000005" iyy="0.007934" iyz="-0.000081" izz="0.015304" />
-    </inertial>
-    <visual>
-      <origin xyz="0 0 0" rpy="0 0 0" />
-      <geometry>
-        <mesh filename="$(find my_arm)/aubo_description/meshes/aubo_i10/visual/link0.DAE" />
-      </geometry>
-      <material name="">
-        <color rgba="1 1 1 1" />
-      </material>
-    </visual>
-    <collision>
-      <origin xyz="0 0 0" rpy="0 0 0" />
-      <geometry>
-        <mesh filename="$(find my_arm)/aubo_description/meshes/aubo_i10/collision/link0.STL" />
-      </geometry>
-    </collision>
-  </link>
-  <link name="shoulder_Link">
-    <inertial>
-      <origin xyz="-0.000004 0.005112 -0.026275" rpy="0 0 0" />
-      <mass value="10.180139" />
-      <inertia ixx="0.043326" ixy="0.000003" ixz="0.000003" iyy="0.042233" iyz="-0.001767" izz="0.029902" />
-    </inertial>
-    <visual>
-      <origin xyz="0 0 0" rpy="0 0 0" />
-      <geometry>
-        <mesh filename="$(find my_arm)/aubo_description/meshes/aubo_i10/visual/link1.DAE" />
-      </geometry>
-      <material name="">
-        <color rgba="0.89804 0.91765 0.92941 1" />
-      </material>
-    </visual>
-    <collision>
-      <origin xyz="0 0 0" rpy="0 0 0" />
-      <geometry>
-        <mesh filename="$(find my_arm)/aubo_description/meshes/aubo_i10/collision/link1.STL" />
-      </geometry>
-    </collision>
-  </link>
-  <joint name="shoulder_joint" type="revolute">
-    <origin xyz="0 0 0.1632" rpy="0 0 3.1415926535897932384626433832795" />
-    <parent link="base_link" />
-    <child link="shoulder_Link" />
-    <axis xyz="0 0 1" />
-    <limit lower="-6.283185307179586476925286766559" upper="6.283185307179586476925286766559" effort="267" start_stop="411" velocity="3.1416" />
-  </joint>
-  <link name="upperArm_Link">
-    <inertial>
-      <origin xyz="0.231117 -0.000013 -0.022852" rpy="0 0 0" />
-      <mass value="18.096361" />
-      <inertia ixx="0.064904" ixy="0.00003" ixz="-0.033711" iyy="1.524623" iyz="0.000015" izz="1.505664" />
-    </inertial>
-    <visual>
-      <origin xyz="0 0 0" rpy="0 0 0" />
-      <geometry>
-        <mesh filename="$(find my_arm)/aubo_description/meshes/aubo_i10/visual/link2.DAE" />
-      </geometry>
-      <material name="">
-        <color rgba="0.89804 0.91765 0.92941 1" />
-      </material>
-    </visual>
-    <collision>
-      <origin xyz="0 0 0" rpy="0 0 0" />
-      <geometry>
-        <mesh filename="$(find my_arm)/aubo_description/meshes/aubo_i10/collision/link2.STL" />
-      </geometry>
-    </collision>
-  </link>
-  <joint name="upperArm_joint" type="revolute">
-    <origin xyz="0 0.2013 0" rpy="-1.5707963267948966192313216916398 -1.5707963267948966192313216916398 0" />
-    <parent link="shoulder_Link" />
-    <child link="upperArm_Link" />
-    <axis xyz="0 0 1" />
-    <limit lower="-6.283185307179586476925286766559" upper="6.283185307179586476925286766559" effort="267" start_stop="411" velocity="3.1416" />
-  </joint>
-  <link name="foreArm_Link">
-    <inertial>
-      <origin xyz="0.41956 -0.000019 0.118053" rpy="0 0 0" />
-      <mass value="4.448092" />
-      <inertia ixx="0.006799" ixy="0.000016" ixz="0.004004" iyy="0.246194" iyz="0.000005" izz="0.24479" />
-    </inertial>
-    <visual>
-      <origin xyz="0 0 0" rpy="0 0 0" />
-      <geometry>
-        <mesh filename="$(find my_arm)/aubo_description/meshes/aubo_i10/visual/link3.DAE" />
-      </geometry>
-      <material name="">
-        <color rgba="1 1 1 1" />
-      </material>
-    </visual>
-    <collision>
-      <origin xyz="0 0 0" rpy="0 0 0" />
-      <geometry>
-        <mesh filename="$(find my_arm)/aubo_description/meshes/aubo_i10/collision/link3.STL" />
-      </geometry>
-    </collision>
-  </link>
-  <joint name="foreArm_joint" type="revolute">
-    <origin xyz="0.647 0 0" rpy="-3.1415926535897932384626433832795 0 0" />
-    <parent link="upperArm_Link" />
-    <child link="foreArm_Link" />
-    <axis xyz="0 0 1" />
-    <limit lower="-6.283185307179586476925286766559" upper="6.283185307179586476925286766559" effort="133" start_stop="207" velocity="2.5656" />
-  </joint>
-  <link name="wrist1_Link">
-    <inertial>
-      <origin xyz="0.000047 0.009773 -0.005726" rpy="0 0 0" />
-      <mass value="1.79166" />
-      <inertia ixx="0.002457" ixy="0.000004" ixz="0.000001" iyy="0.00159" iyz="-0.000123" izz="0.002183" />
-    </inertial>
-    <visual>
-      <origin xyz="0 0 0" rpy="0 0 0" />
-      <geometry>
-        <mesh filename="$(find my_arm)/aubo_description/meshes/aubo_i10/visual/link4.DAE" />
-      </geometry>
-      <material name="">
-        <color rgba="1 1 1 1" />
-      </material>
-    </visual>
-    <collision>
-      <origin xyz="0 0 0" rpy="0 0 0" />
-      <geometry>
-        <mesh filename="$(find my_arm)/aubo_description/meshes/aubo_i10/collision/link4.STL" />
-      </geometry>
-    </collision>
-  </link>
-  <joint name="wrist1_joint" type="revolute">
-    <origin xyz="0.6005 0 0" rpy="3.1415926535897932384626433832795 0 1.5707963267948966192313216916398" />
-    <parent link="foreArm_Link" />
-    <child link="wrist1_Link" />
-    <axis xyz="0 0 1" />
-    <limit lower="-6.283185307179586476925286766559" upper="6.283185307179586476925286766559" effort="49" start_stop="66" velocity="3.1416" />
-  </joint>
-  <link name="wrist2_Link">
-    <inertial>
-      <origin xyz="-0.000038 -0.011278 -0.001539" rpy="0 0 0" />
-      <mass value="1.628022" />
-      <inertia ixx="0.001951" ixy="0.000003" ixz="-0.000001" iyy="0.001154" iyz="0.000042" izz="0.001931" />
-    </inertial>
-    <visual>
-      <origin xyz="0 0 0" rpy="0 0 0" />
-      <geometry>
-        <mesh filename="$(find my_arm)/aubo_description/meshes/aubo_i10/visual/link5.DAE" />
-      </geometry>
-      <material name="">
-        <color rgba="1 1 1 1" />
-      </material>
-    </visual>
-    <collision>
-      <origin xyz="0 0 0" rpy="0 0 0" />
-      <geometry>
-        <mesh filename="$(find my_arm)/aubo_description/meshes/aubo_i10/collision/link5.STL" />
-      </geometry>
-    </collision>
-  </link>
-  <joint name="wrist2_joint" type="revolute">
-    <origin xyz="0 0.1025 0" rpy="-1.5707963267948966192313216916398 0 0" />
-    <parent link="wrist1_Link" />
-    <child link="wrist2_Link" />
-    <axis xyz="0 0 1" />
-    <limit lower="-6.283185307179586476925286766559" upper="6.283185307179586476925286766559" effort="13.5" start_stop="34" velocity="3.1416" />
-  </joint>
-  <link name="wrist3_Link">
-    <inertial>
-      <origin xyz="0.000022 0.0006 -0.017081" rpy="0 0 0" />
-      <mass value="0.1978" />
-      <inertia ixx="0.000118" ixy="0" ixz="0" iyy="0.000112" iyz="0.000001" izz="0.000184" />
-    </inertial>
-    <visual>
-      <origin xyz="0 0 0" rpy="0 0 0" />
-      <geometry>
-        <mesh filename="$(find my_arm)/aubo_description/meshes/aubo_i10/visual/link6.DAE" />
-      </geometry>
-      <material name="">
-        <color rgba="1 1 1 1" />
-      </material>
-    </visual>
-    <collision>
-      <origin xyz="0 0 0" rpy="0 0 0" />
-      <geometry>
-        <mesh filename="$(find my_arm)/aubo_description/meshes/aubo_i10/collision/link6.STL" />
-      </geometry>
-    </collision>
-  </link>
-  <joint name="wrist3_joint" type="revolute">
-    <origin xyz="0 -0.094 0" rpy="1.5707963267948966192313216916398 0 0" />
-    <parent link="wrist2_Link" />
-    <child link="wrist3_Link" />
-    <axis xyz="0 0 1" />
-    <limit lower="-6.283185307179586476925286766559" upper="6.283185307179586476925286766559" effort="13.5" start_stop="34" velocity="3.1416" />
-  </joint>
-  <link name="world" />
-  <joint name="world_joint" type="fixed">
-    <parent link="world" />
-    <child link = "base_link" />
-    <origin xyz="0.0 0.0 0.0" rpy="0.0 0.0 0.0" />
-  </joint>
+    xmlns:xacro="http://wiki.ros.org/xacro">
+    <dh_type type="modified"/>
+    <safety_para singularity_consistent="0.02 0.01 10 0.2 0.045 10"/>
+    <friction_coeff value="0.65"/>
+    <link name="base_link">
+        <inertial>
+            <origin xyz="0.000136 0.001601 0.018986" rpy="0 0 0" />
+            <mass value="2.592" />
+            <inertia ixx="0.008524" ixy="-0.000001" ixz="-0.000005" iyy="0.007934" iyz="-0.000081" izz="0.015304" />
+        </inertial>
+        <visual>
+            <origin xyz="0 0 0" rpy="0 0 0" />
+            <geometry>
+                <mesh filename="file://$(find my_arm)/meshes/aubo_i10/visual/link0.DAE" />
+            </geometry>
+            <material name="">
+                <color rgba="1 1 1 1" />
+            </material>
+        </visual>
+        <collision>
+            <origin xyz="0 0 0" rpy="0 0 0" />
+            <geometry>
+                <mesh filename="file://$(find my_arm)/meshes/aubo_i10/collision/link0.STL" />
+            </geometry>
+        </collision>
+    </link>
+    <link name="shoulder_Link">
+        <inertial>
+            <origin xyz="-0.000004 0.005112 -0.026275" rpy="0 0 0" />
+            <mass value="10.180139" />
+            <inertia ixx="0.043326" ixy="0.000003" ixz="0.000003" iyy="0.042233" iyz="-0.001767" izz="0.029902" />
+        </inertial>
+        <visual>
+            <origin xyz="0 0 0" rpy="0 0 0" />
+            <geometry>
+                <mesh filename="file://$(find my_arm)/meshes/aubo_i10/visual/link1.DAE" />
+            </geometry>
+            <material name="">
+                <color rgba="0.89804 0.91765 0.92941 1" />
+            </material>
+        </visual>
+        <collision>
+            <origin xyz="0 0 0" rpy="0 0 0" />
+            <geometry>
+                <mesh filename="file://$(find my_arm)/meshes/aubo_i10/collision/link1.STL" />
+            </geometry>
+        </collision>
+    </link>
+    <joint name="shoulder_joint" type="revolute">
+        <origin xyz="0 0 0.1632" rpy="0 0 3.1415926535897932384626433832795" />
+        <parent link="base_link" />
+        <child link="shoulder_Link" />
+        <axis xyz="0 0 1" />
+        <limit lower="-6.283185307179586476925286766559" upper="6.283185307179586476925286766559" effort="267" start_stop="411" velocity="3.1416" />
+    </joint>
+    <link name="upperArm_Link">
+        <inertial>
+            <origin xyz="0.231117 -0.000013 -0.022852" rpy="0 0 0" />
+            <mass value="18.096361" />
+            <inertia ixx="0.064904" ixy="0.00003" ixz="-0.033711" iyy="1.524623" iyz="0.000015" izz="1.505664" />
+        </inertial>
+        <visual>
+            <origin xyz="0 0 0" rpy="0 0 0" />
+            <geometry>
+                <mesh filename="file://$(find my_arm)/meshes/aubo_i10/visual/link2.DAE" />
+            </geometry>
+            <material name="">
+                <color rgba="0.89804 0.91765 0.92941 1" />
+            </material>
+        </visual>
+        <collision>
+            <origin xyz="0 0 0" rpy="0 0 0" />
+            <geometry>
+                <mesh filename="file://$(find my_arm)/meshes/aubo_i10/collision/link2.STL" />
+            </geometry>
+        </collision>
+    </link>
+    <joint name="upperArm_joint" type="revolute">
+        <origin xyz="0 0.2013 0" rpy="-1.5707963267948966192313216916398 -1.5707963267948966192313216916398 0" />
+        <parent link="shoulder_Link" />
+        <child link="upperArm_Link" />
+        <axis xyz="0 0 1" />
+        <limit lower="-6.283185307179586476925286766559" upper="6.283185307179586476925286766559" effort="267" start_stop="411" velocity="3.1416" />
+    </joint>
+    <link name="foreArm_Link">
+        <inertial>
+            <origin xyz="0.41956 -0.000019 0.118053" rpy="0 0 0" />
+            <mass value="4.448092" />
+            <inertia ixx="0.006799" ixy="0.000016" ixz="0.004004" iyy="0.246194" iyz="0.000005" izz="0.24479" />
+        </inertial>
+        <visual>
+            <origin xyz="0 0 0" rpy="0 0 0" />
+            <geometry>
+                <mesh filename="file://$(find my_arm)/meshes/aubo_i10/visual/link3.DAE" />
+            </geometry>
+            <material name="">
+                <color rgba="1 1 1 1" />
+            </material>
+        </visual>
+        <collision>
+            <origin xyz="0 0 0" rpy="0 0 0" />
+            <geometry>
+                <mesh filename="file://$(find my_arm)/meshes/aubo_i10/collision/link3.STL" />
+            </geometry>
+        </collision>
+    </link>
+    <joint name="foreArm_joint" type="revolute">
+        <origin xyz="0.647 0 0" rpy="-3.1415926535897932384626433832795 0 0" />
+        <parent link="upperArm_Link" />
+        <child link="foreArm_Link" />
+        <axis xyz="0 0 1" />
+        <limit lower="-6.283185307179586476925286766559" upper="6.283185307179586476925286766559" effort="133" start_stop="207" velocity="2.5656" />
+    </joint>
+    <link name="wrist1_Link">
+        <inertial>
+            <origin xyz="0.000047 0.009773 -0.005726" rpy="0 0 0" />
+            <mass value="1.79166" />
+            <inertia ixx="0.002457" ixy="0.000004" ixz="0.000001" iyy="0.00159" iyz="-0.000123" izz="0.002183" />
+        </inertial>
+        <visual>
+            <origin xyz="0 0 0" rpy="0 0 0" />
+            <geometry>
+                <mesh filename="file://$(find my_arm)/meshes/aubo_i10/visual/link4.DAE" />
+            </geometry>
+            <material name="">
+                <color rgba="1 1 1 1" />
+            </material>
+        </visual>
+        <collision>
+            <origin xyz="0 0 0" rpy="0 0 0" />
+            <geometry>
+                <mesh filename="file://$(find my_arm)/meshes/aubo_i10/collision/link4.STL" />
+            </geometry>
+        </collision>
+    </link>
+    <joint name="wrist1_joint" type="revolute">
+        <origin xyz="0.6005 0 0" rpy="3.1415926535897932384626433832795 0 1.5707963267948966192313216916398" />
+        <parent link="foreArm_Link" />
+        <child link="wrist1_Link" />
+        <axis xyz="0 0 1" />
+        <limit lower="-6.283185307179586476925286766559" upper="6.283185307179586476925286766559" effort="49" start_stop="66" velocity="3.1416" />
+    </joint>
+    <link name="wrist2_Link">
+        <inertial>
+            <origin xyz="-0.000038 -0.011278 -0.001539" rpy="0 0 0" />
+            <mass value="1.628022" />
+            <inertia ixx="0.001951" ixy="0.000003" ixz="-0.000001" iyy="0.001154" iyz="0.000042" izz="0.001931" />
+        </inertial>
+        <visual>
+            <origin xyz="0 0 0" rpy="0 0 0" />
+            <geometry>
+                <mesh filename="file://$(find my_arm)/meshes/aubo_i10/visual/link5.DAE" />
+            </geometry>
+            <material name="">
+                <color rgba="1 1 1 1" />
+            </material>
+        </visual>
+        <collision>
+            <origin xyz="0 0 0" rpy="0 0 0" />
+            <geometry>
+                <mesh filename="file://$(find my_arm)/meshes/aubo_i10/collision/link5.STL" />
+            </geometry>
+        </collision>
+    </link>
+    <joint name="wrist2_joint" type="revolute">
+        <origin xyz="0 0.1025 0" rpy="-1.5707963267948966192313216916398 0 0" />
+        <parent link="wrist1_Link" />
+        <child link="wrist2_Link" />
+        <axis xyz="0 0 1" />
+        <limit lower="-6.283185307179586476925286766559" upper="6.283185307179586476925286766559" effort="13.5" start_stop="34" velocity="3.1416" />
+    </joint>
+    <link name="wrist3_Link">
+        <inertial>
+            <origin xyz="0.000022 0.0006 -0.017081" rpy="0 0 0" />
+            <mass value="0.1978" />
+            <inertia ixx="0.000118" ixy="0" ixz="0" iyy="0.000112" iyz="0.000001" izz="0.000184" />
+        </inertial>
+        <visual>
+            <origin xyz="0 0 0" rpy="0 0 0" />
+            <geometry>
+                <mesh filename="file://$(find my_arm)/meshes/aubo_i10/visual/link6.DAE" />
+            </geometry>
+            <material name="">
+                <color rgba="1 1 1 1" />
+            </material>
+        </visual>
+        <collision>
+            <origin xyz="0 0 0" rpy="0 0 0" />
+            <geometry>
+                <mesh filename="file://$(find my_arm)/meshes/aubo_i10/collision/link6.STL" />
+            </geometry>
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