Commit message: 实现启动gazebo仿真

File: urdf/aubo_i10.ros2_control.xacro (robot description, xacro)
@@ -49,15 +49,28 @@
                 <state_interface name="velocity"/>
             </joint>
+            <joint name="panda_hand_joint" type="fixed">
+                <parent link="wrist3_Link" />
+                <child link="panda_hand" />
+                <origin rpy="0 0 0" xyz="0 0 0.01" />
+            </joint>
             <joint name="panda_finger_joint1">
                 <command_interface name="position"/>
                 <state_interface name="position">
-                    <param name="initial_value">${initial_positions['panda_finger_joint1']}</param>
+                    <param name="initial_value">0.0</param>
                 </state_interface>
                 <state_interface name="velocity"/>
             </joint>
+            <!-- <joint name="panda_finger_joint2">
+                <param name="mimic">panda_finger_joint1</param>
+                <command_interface name="position"/>
+                <state_interface name="position">
+                    <param name="initial_value">0.0</param>
+                </state_interface>
+                <state_interface name="velocity"/>
+            </joint> -->
         </ros2_control>
         <gazebo>
             <plugin filename="libgazebo_ros2_control.so" name="gazebo_ros2_control">
-                <parameters>file://$(find my_arm)/config/ros2_controllers.yaml</parameters>
+                <parameters>$(find my_arm)/config/ros2_controllers.yaml</parameters>
             </plugin>
         </gazebo>

File: urdf/aubo_i10.urdf.xacro (robot description, xacro)
@@ -201,61 +201,94 @@
         <limit lower="-6.283185307179586476925286766559" upper="6.283185307179586476925286766559" effort="13.5" start_stop="34" velocity="3.1416" />
     </joint>
+    <!-- panda_hand -->
+    <joint name="panda_hand_joint" type="fixed">
+        <parent link="wrist3_Link"/>
+        <child link="panda_hand"/>
+        <origin rpy="0 0 0" xyz="0 0 0"/>
+    </joint>
     <link name="panda_hand">
-        <visual>
-            <geometry>
-                <mesh filename="file://$(find my_arm)/meshes/aubo_i10/visual/hand.dae" />
-            </geometry>
-        </visual>
-        <collision>
-            <geometry>
-                <mesh filename="file://$(find my_arm)/meshes/aubo_i10/collision/hand.stl" />
-            </geometry>
-        </collision>
-    </link>
-    <joint name="panda_hand_joint" type="fixed">
-        <parent link="wrist3_Link" />
-        <child link="panda_hand" />
-        <origin rpy="0 0 0" xyz="0 0 0.01" />
-    </joint>
+        <inertial>
+            <mass value="0.73"/>
+            <origin rpy="0 0 0" xyz="0 0.0015244 0.0275912"/>
+            <inertia ixx="0.00278560230025" ixy="0.0" ixz="0.0" iyy="0.000400033405336" iyz="0.0" izz="0.00256378041832"/>
+        </inertial>
+        <visual>
+            <origin rpy="0 0 0" xyz="0 0 0"/>
+            <geometry>
+                <mesh filename="file://$(find my_arm)/meshes/aubo_i10/visual/hand.dae"/>
+            </geometry>
+            <material name="">
+                <color rgba="1 1 1 1"/>
+            </material>
+        </visual>
+        <collision>
+            <origin rpy="0 0 0" xyz="0 0 0"/>
+            <geometry>
+                <mesh filename="file://$(find my_arm)/meshes/aubo_i10/collision/hand.stl"/>
+            </geometry>
+        </collision>
+    </link>
+    <!-- panda_leftfinger -->
     <link name="panda_leftfinger">
-        <visual>
-            <geometry>
-                <mesh filename="file://$(find my_arm)/meshes/aubo_i10/visual/finger.dae" />
-            </geometry>
-        </visual>
-        <collision>
-            <geometry>
-                <mesh filename="file://$(find my_arm)/meshes/aubo_i10/collision/finger.stl" />
+        <inertial>
+            <mass value="0.1"/>
+            <origin rpy="0 0 0" xyz="0 0.0145644 0.0227941"/>
+            <inertia ixx="3.01220925051e-05" ixy="0.0" ixz="0.0" iyy="2.95873808038e-05" iyz="0.0" izz="6.95125211657e-06"/>
+        </inertial>
+        <visual>
+            <origin rpy="0 0 0" xyz="0 0 0"/>
+            <geometry>
+                <mesh filename="file://$(find my_arm)/meshes/aubo_i10/visual/finger.dae"/>
+            </geometry>
+            <material name="">
+                <color rgba="1 1 1 1"/>
+            </material>
+        </visual>
+        <collision>
+            <origin rpy="0 0 0" xyz="0 0 0"/>
+            <geometry>
+                <mesh filename="file://$(find my_arm)/meshes/aubo_i10/collision/finger.stl"/>
+            </geometry>
+        </collision>
+    </link>
+    <!-- panda_rightfinger -->
+    <link name="panda_rightfinger">
+        <inertial>
+            <mass value="0.1"/>
+            <origin rpy="0 0 3.14159265359" xyz="0 0.0145644 0.0227941"/>
+            <inertia ixx="3.01220925051e-05" ixy="0.0" ixz="0.0" iyy="2.95873808038e-05" iyz="0.0" izz="6.95125211657e-06"/>
+        </inertial>
+        <visual>
+            <origin rpy="0 0 3.14159265359" xyz="0 0 0"/>
+            <geometry>
+                <mesh filename="file://$(find my_arm)/meshes/aubo_i10/visual/finger.dae"/>
+            </geometry>
+            <material name="">
+                <color rgba="1 1 1 1"/>
+            </material>
+        </visual>
+        <collision>
+            <origin rpy="0 0 3.14159265359" xyz="0 0 0"/>
+            <geometry>
+                <mesh filename="file://$(find my_arm)/meshes/aubo_i10/collision/finger.stl"/>
             </geometry>
         </collision>
     </link>
     <joint name="panda_finger_joint1" type="prismatic">
-        <parent link="panda_hand" />
-        <child link="panda_leftfinger" />
-        <origin rpy="0 0 0" xyz="0 0 0.0584" />
-        <axis xyz="0 1 0" />
-        <limit effort="20" lower="0.0" upper="0.04" velocity="0.2" />
-    </joint>
-    <link name="panda_rightfinger">
-        <visual>
-            <origin rpy="0 0 3.14159265359" xyz="0 0 0" />
-            <geometry>
-                <mesh filename="file://$(find my_arm)/meshes/aubo_i10/visual/finger.dae" />
-            </geometry>
-        </visual>
-        <collision>
-            <origin rpy="0 0 3.14159265359" xyz="0 0 0" />
-            <geometry>
-                <mesh filename="file://$(find my_arm)/meshes/aubo_i10/collision/finger.stl" />
-            </geometry>
-        </collision>
-    </link>
+        <parent link="panda_hand"/>
+        <child link="panda_leftfinger"/>
+        <origin rpy="0 0 0" xyz="0 0 0.0584"/>
+        <axis xyz="0 1 0"/>
+        <limit effort="20" lower="-0.001" upper="0.04" velocity="0.3"/>
+        <dynamics damping="1.0" friction="1.0"/>
+    </joint>
     <joint name="panda_finger_joint2" type="prismatic">
-        <parent link="panda_hand" />
-        <child link="panda_rightfinger" />
-        <origin rpy="0 0 0" xyz="0 0 0.0584" />
-        <axis xyz="0 -1 0" />
-        <limit effort="20" lower="0.0" upper="0.04" velocity="0.2" />
-        <mimic joint="panda_finger_joint1" />
+        <mimic joint="panda_finger_joint1" multiplier="-1.0" offset="0" />
+        <parent link="panda_hand"/>
+        <child link="panda_rightfinger"/>
+        <origin rpy="0 0 0" xyz="0 0 0.0584"/>
+        <axis xyz="0 -1 0"/>
+        <limit effort="20" lower="-0.001" upper="0.04" velocity="0.3"/>
+        <dynamics damping="1.0" friction="1.0"/>
     </joint>
     <link name="world" />

Commit message: 启用panda_finger_joint2关节的控制接口

File: urdf/aubo_i10.ros2_control.xacro (robot description, xacro)
@@ -61,5 +61,5 @@
                 <state_interface name="velocity"/>
             </joint>
-            <!-- <joint name="panda_finger_joint2">
+            <joint name="panda_finger_joint2">
                 <param name="mimic">panda_finger_joint1</param>
                 <command_interface name="position"/>
@@ -68,5 +68,5 @@
                 </state_interface>
                 <state_interface name="velocity"/>
-            </joint> -->
+            </joint>
         </ros2_control>
         <gazebo>

Commit message: 在配置文件中启用panda_finger_joint2关节控制，并移除相关的mimic参数

File: urdf/aubo_i10.ros2_control.xacro (robot description, xacro)
@@ -62,5 +62,6 @@
             </joint>
             <joint name="panda_finger_joint2">
-                <param name="mimic">panda_finger_joint1</param>
+                <!-- <param name="mimic">panda_finger_joint1</param>
+                <param name="multiplier">-1.0</param> -->
                 <command_interface name="position"/>
                 <state_interface name="position">

File: urdf/aubo_i10.urdf.xacro (robot description, xacro)
@@ -284,5 +284,5 @@
     </joint>
     <joint name="panda_finger_joint2" type="prismatic">
-        <mimic joint="panda_finger_joint1" multiplier="-1.0" offset="0" />
+        <!-- <mimic joint="panda_finger_joint1" multiplier="-1.0" offset="0" /> -->
         <parent link="panda_hand"/>
         <child link="panda_rightfinger"/>
